File: elec/layout/default/lv2842xlvddcr.kicad_pcb (KiCad board)
At the start: 2 copper layers, 225.7 x 100.8 mm, 8 parts

Commit message: Remove xmas crud
Other:
- board outline removed
- board text removed: "{{GITHASH}}"
