File: elec/layout/test-1v8/test-1v8.kicad_pcb (KiCad board)
At the start: 2 copper layers, 8 parts, among them U3 10µH ±20%

Commit message: build with latest
Connections:
- C2 pad 1: hv-1 -> hv
- C3 pad 1: hv -> hv-1
- R2 pad 1: hv -> hv-1
- U2 pad 4: hv-1 -> hv
- U2 pad 5: hv-1 -> hv
- U3 pad 2: hv -> hv-1
Changed lines of the file:
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@@
     (net 2 "FB")
     (net 3 "SW")
-    (net 4 "hv-1")
+    (net 4 "hv")
     (net 5 "CB")
     (net 6 "gnd")
-    (net 7 "hv")
+    (net 7 "hv-1")
     (footprint "atopile:C0402-b3ef17"
         (layer "F.Cu")
@@
             (size 1.41 1.35)
             (layers "F.Cu" "F.Mask" "F.Paste")
-            (net 7 "hv")
+            (net 7 "hv-1")
         )
         (pad "2" smd rect
@@
             (size 1.6 3.5)
             (layers "F.Cu" "F.Mask" "F.Paste")
-            (net 7 "hv")
+            (net 7 "hv-1")
         )
         (embedded_fonts no)
@@
             (size 1.41 1.35)
             (layers "F.Cu" "F.Mask" "F.Paste")
-            (net 4 "hv-1")
+            (net 4 "hv")
         )
         (pad "2" smd rect
@@
             (size 0.57 0.54)
             (layers "F.Cu" "F.Mask" "F.Paste")
-            (net 7 "hv")
+            (net 7 "hv-1")
         )
         (pad "2" smd rect
@@
             (size 1.1 0.6)
             (layers "F.Cu" "F.Mask" "F.Paste")
-            (net 4 "hv-1")
+            (net 4 "hv")
         )
         (pad "5" smd rect
@@
             (size 1.1 0.6)
             (layers "F.Cu" "F.Mask" "F.Paste")
-            (net 4 "hv-1")
+            (net 4 "hv")
         )
         (pad "6" smd rect
