File: elec/layout/test-3v3/test-3v3.kicad_pcb (KiCad board)
At the start: 2 copper layers, 8 parts, among them U3 10µH ±20%

Commit message: build with latest
Connections:
- net cathode renamed SW
Changed lines of the file:
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@@
     (net 2 "gnd-1")
     (net 3 "hv")
-    (net 4 "cathode")
+    (net 4 "SW")
     (net 5 "CB")
     (net 6 "gnd")
@@
             (size 1.6 3.5)
             (layers "F.Cu" "F.Mask" "F.Paste")
-            (net 4 "cathode")
+            (net 4 "SW")
         )
         (pad "2" smd rect
@@
             (size 0.79 0.54)
             (layers "F.Cu" "F.Mask" "F.Paste")
-            (net 4 "cathode")
+            (net 4 "SW")
         )
         (embedded_fonts no)
@@
             (size 1 0.75)
             (layers "F.Cu" "F.Mask" "F.Paste")
-            (net 4 "cathode")
+            (net 4 "SW")
         )
         (pad "2" smd rect
@@
             (size 1.1 0.6)
             (layers "F.Cu" "F.Mask" "F.Paste")
-            (net 4 "cathode")
+            (net 4 "SW")
         )
         (embedded_fonts no)
