File: elec/layout/test-8v/test-8v.kicad_pcb (KiCad board)
At the start: 2 copper layers, 8 parts, among them U3 10µH ±20%

Commit message: build with latest
Connections:
- net SW renamed cathode
- C2 pad 2: gnd-1 -> gnd
- C3 pad 2: gnd -> gnd-1
- R1 pad 2: gnd -> gnd-1
- U1 pad 2: gnd -> gnd-1
- U2 pad 2: gnd-1 -> gnd
Changed lines of the file:
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@@
     (net 0 "")
     (net 1 "hv")
-    (net 2 "gnd-1")
+    (net 2 "gnd")
     (net 3 "FB")
     (net 4 "CB")
     (net 5 "hv-1")
-    (net 6 "SW")
-    (net 7 "gnd")
+    (net 6 "cathode")
+    (net 7 "gnd-1")
     (footprint "atopile:C0402-b3ef17"
         (layer "F.Cu")
@@
             (size 0.79 0.54)
             (layers "F.Cu" "F.Mask" "F.Paste")
-            (net 6 "SW")
+            (net 6 "cathode")
         )
         (embedded_fonts no)
@@
             (size 1 0.75)
             (layers "F.Cu" "F.Mask" "F.Paste")
-            (net 6 "SW")
+            (net 6 "cathode")
         )
         (pad "2" smd rect
@@
             (size 1 0.75)
             (layers "F.Cu" "F.Mask" "F.Paste")
-            (net 7 "gnd")
+            (net 7 "gnd-1")
         )
         (embedded_fonts no)
@@
             (size 1.41 1.35)
             (layers "F.Cu" "F.Mask" "F.Paste")
-            (net 7 "gnd")
+            (net 7 "gnd-1")
         )
         (embedded_fonts no)
@@
             (size 0.57 0.54)
             (layers "F.Cu" "F.Mask" "F.Paste")
-            (net 7 "gnd")
+            (net 7 "gnd-1")
         )
         (embedded_fonts no)
@@
             (size 1.41 1.35)
             (layers "F.Cu" "F.Mask" "F.Paste")
-            (net 2 "gnd-1")
+            (net 2 "gnd")
         )
         (embedded_fonts no)
@@
             (size 1.6 3.5)
             (layers "F.Cu" "F.Mask" "F.Paste")
-            (net 6 "SW")
+            (net 6 "cathode")
         )
         (pad "2" smd rect
@@
             (size 1.1 0.6)
             (layers "F.Cu" "F.Mask" "F.Paste")
-            (net 2 "gnd-1")
+            (net 2 "gnd")
         )
         (pad "3" smd rect
@@
             (size 1.1 0.6)
             (layers "F.Cu" "F.Mask" "F.Paste")
-            (net 6 "SW")
+            (net 6 "cathode")
         )
         (embedded_fonts no)
